File: motherboard.brd (EAGLE design)
At the start: 152.4 x 101.6 mm, 61 parts, among them U1 A13, Y1 24MHz

Commit message: The feverdream continues unabated.
Routing:
- net 1.5V: track 20.2 -> 22.4 mm, vias 10 -> 14
- net GND: track 19.0 -> 20.1 mm, vias 7 -> 9
- net DDR_CK_P: track 0.00 -> 0.57 mm, vias 0 -> 1
- net DDR_A8: track 0.00 -> 0.57 mm, vias 0 -> 1
- net DDR_A11: track 0.00 -> 0.57 mm, vias 0 -> 1
- net DDR_DQS1_N: track 0.00 -> 0.57 mm, vias 0 -> 1
- net DDR_A6: track 0.00 -> 0.57 mm, vias 0 -> 1
- net DDR_D5: track 0.00 -> 0.57 mm, vias 0 -> 1
- net DDR_DQS1_P: track 0.00 -> 0.57 mm, vias 0 -> 1
- net DDR_CKE: track 0.00 -> 0.54 mm, vias 0 -> 1
- net DDR_CK_N: track 0.13 -> 0.57 mm, vias 0 -> 1
Other:
- board text added: "FeverDream"
